Commit message: re-try simulation

File: social_costmap_ws/src/turtlebot3/turtlebot3_description/urdf/turtlebot3_waffle_pi.urdf (robot description, URDF)
Before this commit: robot turtlebot3_waffle_pi, 11 links, 10 joints
Links:
- removed link base_scan
- added link base_laser, mass 0.114; collision cylinder length=0.0315 radius=0.055; visual mesh filename=package://turtlebot3_description/meshes/sensors/lds.stl scale=0.001 0.001 0.001
Joints:
- joint scan_joint: child base_scan -> base_laser
